File: tesis/esquematicos/medicion_fg/medicion_fg.sch (KiCad schematic (older format))
At the start: 9 parts, among them K220 ISrc, K617 Chargemeter

Commit message: Abrir esquematico con Kicad nuevo
Parts:
- added Cfg?, Cinyector?: C, symbol C-RESCUE-medicion_fg
- added Ddrain?, Dinyector?, Dlector?: DIODE, symbol DIODE
- added K?: ISrc, symbol ISrc
- added K?: Chargemeter, symbol Chargemeter
- added Rpcb?: R, symbol R-RESCUE-medicion_fg
- added U?: Túnel, symbol Túnel
- Cfg, Cinyector: symbol C -> C-RESCUE-medicion_fg
- Rpcb: symbol R -> R-RESCUE-medicion_fg
Connections:
- net FG: now also Cfg?.2, Cinyector?.1, U?.2 (G)
- net Inyector: now also Cinyector?.2, Dinyector?.2 (K), K?.1 (H), Rpcb?.2
- net LectorN: now also Ddrain?.1 (A)
- net LectorP: now also Cfg?.1, Dlector?.2 (K), K?.2 (L), Rpcb?.1
- net Sustrato: now also Dinyector?.1 (A), Dlector?.1 (A), K?.3 (G)
- net at K220.1 (H), K617.2 (L): now also K?.1 (H), K?.2 (L)
- net at Ddrain.2 (K): now also Ddrain?.2 (K)
- net at U?.1 (B): now also U?.1 (B)
Changed lines of the file:
@@
 EESchema Schematic File Version 2
+LIBS:medicion_fg-rescue
 LIBS:power
 LIBS:device
@@
 LIBS:memory
 LIBS:xilinx
-LIBS:special
 LIBS:microcontrollers
 LIBS:dsp
@@
 LIBS:contrib
 LIBS:valves
-LIBS:medicion
 LIBS:medicion_fg-cache
 EELAYER 25 0
@@
 $EndComp
 Wire Wire Line
-	3200 2850 3450 2850
-Wire Wire Line
-	3450 2850 4250 2850
-Wire Wire Line
-	4250 2850 4350 2850
+	3200 2850 4350 2850
 Wire Wire Line
 	4250 2450 4850 2450
 Wire Wire Line
-	4850 2450 4850 2450
-Wire Wire Line
-	4850 2450 4850 3000
+	4850 2050 4850 3000
 Wire Wire Line
 	4850 3000 3050 3000
 $Comp
-L C Cinyector
+L C-RESCUE-medicion_fg Cinyector
 U 1 1 55F85E8C
 P 3650 2450
@@
 $EndComp
 $Comp
-L C Cfg
+L C-RESCUE-medicion_fg Cfg
 U 1 1 55F85ED9
 P 4050 2450
@@
 	4250 2050 4250 2450
 Wire Wire Line
-	3450 2050 3450 2050
+	3050 2050 3600 2050
 Wire Wire Line
 	3450 2050 3450 2450
@@
 	3850 2250 3850 2450
 $Comp
-L R Rpcb
+L R-RESCUE-medicion_fg Rpcb
 U 1 1 55F86C0F
 P 3850 2050
@@
 	0    1    1    0
 $EndComp
-Wire Wire Line
-	3050 2050 3450 2050
-Wire Wire Line
-	3450 2050 3600 2050
 Connection ~ 3450 2050
 Wire Wire Line
@@
 Wire Wire Line
 	3050 2550 3050 2700
-Wire Wire Line
-	4850 2050 4850 2450
 Connection ~ 4850 2450
 Text Label 4350 2450 0    60   ~ 0
+WellLector
+$Comp
+L ISrc K?
+U 1 1 5B787432
+P 3050 2850
+F 0 "K?" H 3200 3000 60  0000 C CNN
+F 1 "ISrc" H 2850 2875 60  0001 C CNN
+F 2 "" H 3050 2850 60  0000 C CNN
+F 3 "" H 3050 2850 60  0000 C CNN
+	1    3050 2850
+	1    0    0    -1
+$EndComp
+$Comp
+L Chargemeter K?
+U 1 1 5B787433
+P 3050 2400
+F 0 "K?" H 3200 2550 60  0000 C CNN
+F 1 "Chargemeter" H 3050 2400 60  0001 C CNN
+F 2 "" H 3050 2400 60  0000 C CNN
+F 3 "" H 3050 2400 60  0000 C CNN
+	1    3050 2400
+	1    0    0    -1
+$EndComp
+$Comp
+L DIODE Dinyector?
+U 1 1 5B787434
+P 3450 2650
+F 0 "Dinyector?" H 3450 2750 40  0000 C CNN
+F 1 "DIODE" H 3450 2550 40  0001 C CNN
+F 2 "" H 3450 2650 60  0000 C CNN
+F 3 "" H 3450 2650 60  0000 C CNN
+	1    3450 2650
+	0    -1   -1   0
+$EndComp
+$Comp
+L DIODE Dlector?
+U 1 1 5B787435
+P 4250 2650
+F 0 "Dlector?" H 4250 2550 40  0000 C CNN
+F 1 "DIODE" H 4250 2550 40  0001 C CNN
+F 2 "" H 4250 2650 60  0000 C CNN
+F 3 "" H 4250 2650 60  0000 C CNN
+	1    4250 2650
+	0    -1   -1   0
+$EndComp
+Wire Wire Line
+	3200 2850 4350 2850
+Wire Wire Line
+	4250 2450 4850 2450
+Wire Wire Line
+	4850 2050 4850 3000
+Wire Wire Line
+	4850 3000 3050 3000
+$Comp
+L C-RESCUE-medicion_fg Cinyector?
+U 1 1 5B787436
+P 3650 2450
+F 0 "Cinyector?" V 3800 2350 40  0000 L CNN
+F 1 "C" H 3656 2365 40  0001 L CNN
+F 2 "" H 3688 2300 30  0000 C CNN
+F 3 "" H 3650 2450 60  0000 C CNN
+	1    3650 2450
+	0    1    1    0
+$EndComp
+$Comp
+L C-RESCUE-medicion_fg Cfg?
+U 1 1 5B787437
+P 4050 2450
+F 0 "Cfg?" V 4200 2400 40  0000 L CNN
+F 1 "C" H 4056 2365 40  0001 L CNN
+F 2 "" H 4088 2300 30  0000 C CNN
+F 3 "" H 4050 2450 60  0000 C CNN
+	1    4050 2450
+	0    1    1    0
+$EndComp
+Text HLabel 3050 2050 1    60   Input ~ 0
+Inyector
+Text HLabel 4850 2050 1    60   Input ~ 0
+LectorP
+$Comp
+L DIODE Ddrain?
+U 1 1 5B787438
+P 4500 2250
+F 0 "Ddrain?" H 4500 2350 40  0000 C CNN
+F 1 "DIODE" H 4500 2150 40  0001 C CNN
+F 2 "" H 4500 2250 60  0000 C CNN
+F 3 "" H 4500 2250 60  0000 C CNN
+	1    4500 2250
+	0    1    1    0
+$EndComp
+Text HLabel 4500 2050 1    60   Input ~ 0
+LectorN
+Wire Wire Line
+	4250 2050 4250 2450
+Wire Wire Line
+	3050 2050 3600 2050
+Wire Wire Line
+	3450 2050 3450 2450
+Text HLabel 4350 2850 2    60   Input ~ 0
+Sustrato
+Connection ~ 4250 2850
+$Comp
+L Túnel U?
+U 1 1 5B787439
+P 3650 2250
+F 0 "U?" H 3650 2350 60  0001 C CNN
+F 1 "Túnel" H 3650 2150 60  0001 C CNN
+F 2 "" H 3650 2250 60  0000 C CNN
+F 3 "" H 3650 2250 60  0000 C CNN
+	1    3650 2250
+	1    0    0    -1
+$EndComp
+Wire Wire Line
+	3850 2250 3850 2450
+$Comp
+L R-RESCUE-medicion_fg Rpcb?
+U 1 1 5B78743A
+P 3850 2050
+F 0 "Rpcb?" V 3850 2050 40  0000 C CNN
+F 1 "R" V 3857 2051 40  0001 C CNN
+F 2 "" V 3780 2050 30  0000 C CNN
+F 3 "" H 3850 2050 30  0000 C CNN
+	1    3850 2050
+	0    1    1    0
+$EndComp
+Connection ~ 3450 2050
+Wire Wire Line
+	4100 2050 4250 2050
+Text Label 3850 2400 0    60   ~ 0
+FG
+Connection ~ 3450 2850
+Wire Wire Line
+	3050 2250 3050 2050
+Wire Wire Line
+	3050 2550 3050 2700
+Connection ~ 4850 2450
+Text Label 4350 2450 0    60   ~ 0
